File: PCB/fan4.kicad_sch (KiCad schematic)
At the start: 5 parts, among them J4 Conn_01x02, Q4 IRLML0030

Commit message: finished PCB
Parts:
- removed Q4: IRLML0030, Package_TO_SOT_SMD:SOT-23, symbol Transistor_FET:IRLML0030
- added Mosfet4: IRLML0030, Package_TO_SOT_SMD:SOT-23, symbol Transistor_FET:IRLML0030
- J4: value Conn_01x02 -> Fan 4
- R7, R8: value R -> 100k
Connections:
- net +12V: now also D4.1 (K), J4.1 (Pin_1); no longer J4.2 (Pin_2)
- net GND: now also R8.2, Mosfet4.2 (S); no longer R7.2
- net at R8.1: now also R7.2, Mosfet4.1 (G); no longer R7.1
- net Fan4: no longer names the net of D4.2 (A)
- net Fan4: now also J4.2 (Pin_2), Mosfet4.3 (D); no longer D4.1 (K)
- new net Fan 4: R7.1
