File: PCB/FanBoardPCB.kicad_sch (KiCad schematic)
At the start: 0 parts

Commit message: Added Schematic
Not sure if its right tho :0
Parts:
- added C1, C2, C3, C4: 100uF, symbol Device:C
- added D1, D2, D3, D4, D6, D7, D8, D9: D, symbol Device:D
- added D5: LED, symbol Device:LED
- added J1: Fan1, symbol Connector_Generic:Conn_01x02
- added J2: Fan2, symbol Connector_Generic:Conn_01x02
- added J3: Fan3, symbol Connector_Generic:Conn_01x02
- added J4: Fan4, symbol Connector_Generic:Conn_01x02
- added J5: FanBoardController, symbol Connector_Generic:Conn_02x03_Top_Bottom
- added Q1, Q2, Q3, Q4: IRLML0030, Package_TO_SOT_SMD:SOT-23, symbol Transistor_FET:IRLML0030
- added R1, R2, R3, R4, R5, R6, R7, R8: 100k, symbol Device:R_US
- added R9: 1k, symbol Device:R_US
Connections:
- new net: Q1.1 (G), R2.2
- new net: D4.1 (K), D6.1 (K), J4.2 (Pin_2)
- new net: C3.1, C4.1
- new net: D1.1 (K), D9.1 (K), J1.2 (Pin_2)
- new net: D3.1 (K), D7.1 (K), J3.2 (Pin_2)
- new net: Q4.1 (G), R8.2
- new net: Q2.1 (G), R4.2
- new net: C1.2, C2.2
- new net: Q3.1 (G), R6.2
- new net: D5.2 (A), R9.2
- new net: D2.1 (K), D8.1 (K), J2.2 (Pin_2)
- new net 12V: C1.1, C2.1, J5.1 (Pin_1), Q1.3 (D), Q2.3 (D), Q3.3 (D), Q4.3 (D), R9.1
- new net FanIn1: J5.2 (Pin_2), R1.1, R2.1
- new net FanIn2: J5.3 (Pin_3), R3.1, R4.1
- new net FanIn3: J5.5 (Pin_5), R5.1, R6.1
- new net FanIn4: J5.6 (Pin_6), R7.1, R8.1
- new net FanOut1: D9.2 (A), Q1.2 (S)
- new net FanOut2: D8.2 (A), Q2.2 (S)
- new net FanOut3: D7.2 (A), Q3.2 (S)
- new net FanOut4: D6.2 (A), Q4.2 (S)
- new net GND: C3.2, C4.2, D1.2 (A), D2.2 (A), D3.2 (A), D4.2 (A), D5.1 (K), J1.1 (Pin_1), J2.1 (Pin_1), J3.1 (Pin_1), J4.1 (Pin_1), J5.4 (Pin_4), R1.2, R3.2, R5.2, R7.2

Commit message: Fixed Sch
Parts:
- removed C3, C4: 100uF, symbol Device:C
- removed D6, D7, D8, D9: D, symbol Device:D
Connections:
- net FanOut1: now also D1.1 (K), J1.2 (Pin_2)
- net FanOut2: now also D2.1 (K), J2.2 (Pin_2)
- net FanOut3: now also D3.1 (K), J3.2 (Pin_2)
- net FanOut4: now also D4.1 (K), J4.2 (Pin_2)
- net GND: now also C1.2, C2.2

Commit message: Started on PCB
Parts:
- C1, C2: footprint (none) -> Capacitor_SMD:C_0805_2012Metric
- D1, D2, D3, D4: footprint (none) -> Diode_SMD:D_0805_2012Metric
- D5: footprint (none) -> LED_SMD:LED_0805_2012Metric
- J1, J2, J3, J4: footprint (none) -> UTSVT_Connectors:Molex_MicroFit3.0_1x2xP3.00mm_PolarizingPeg_Vertical
- J5: footprint (none) -> Connector_Molex:Molex_Micro-Fit_3.0_43650-0615_1x06_P3.00mm_Vertical
- R1, R2, R3, R4, R5, R6, R7, R8, R9: footprint (none) -> Resistor_SMD:R_0805_2012Metric
Changed lines of the file:
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@@
 			)
 		)
-		(property "Footprint" ""
+		(property "Footprint" "Resistor_SMD:R_0805_2012Metric"
 			(at 117.856 120.904 90)
 			(effects
@@
 			)
 		)
-		(property "Footprint" ""
+		(property "Footprint" "Diode_SMD:D_0805_2012Metric"
 			(at 171.45 144.78 0)
 			(effects
@@
 			)
 		)
-		(property "Footprint" ""
+		(property "Footprint" "Resistor_SMD:R_0805_2012Metric"
 			(at 117.856 94.234 90)
 			(effects
@@
 			)
 		)
-		(property "Footprint" ""
+		(property "Footprint" "UTSVT_Connectors:Molex_MicroFit3.0_1x2xP3.00mm_PolarizingPeg_Vertical"
 			(at 161.29 143.51 0)
 			(effects
@@
 			)
 		)
-		(property "Footprint" ""
+		(property "Footprint" "Resistor_SMD:R_0805_2012Metric"
 			(at 122.174 138.684 90)
 			(effects
@@
 			)
 		)
-		(property "Footprint" ""
+		(property "Footprint" "Diode_SMD:D_0805_2012Metric"
 			(at 171.45 80.01 0)
 			(effects
@@
 			)
 		)
-		(property "Footprint" ""
+		(property "Footprint" "Resistor_SMD:R_0805_2012Metric"
 			(at 117.856 145.034 90)
 			(effects
@@
 			)
 		)
-		(property "Footprint" ""
+		(property "Footprint" "Resistor_SMD:R_0805_2012Metric"
 			(at 122.174 87.884 90)
 			(effects
@@
 			)
 		)
-		(property "Footprint" ""
+		(property "Footprint" "Capacitor_SMD:C_0805_2012Metric"
 			(at 84.7852 86.36 0)
 			(effects
@@
 			)
 		)
-		(property "Footprint" ""
+		(property "Footprint" "Connector_Molex:Molex_Micro-Fit_3.0_43650-0615_1x06_P3.00mm_Vertical"
 			(at 173.99 58.42 0)
 			(effects
@@
 			)
 		)
-		(property "Footprint" ""
+		(property "Footprint" "Resistor_SMD:R_0805_2012Metric"
 			(at 122.174 114.554 90)
 			(effects
@@
 			)
 		)
-		(property "Footprint" ""
+		(property "Footprint" "Diode_SMD:D_0805_2012Metric"
 			(at 171.45 123.19 0)
 			(effects
@@
 			)
 		)
-		(property "Footprint" ""
+		(property "Footprint" "UTSVT_Connectors:Molex_MicroFit3.0_1x2xP3.00mm_PolarizingPeg_Vertical"
 			(at 161.29 121.92 0)
 			(effects
@@
 			)
 		)
-		(property "Footprint" ""
+		(property "Footprint" "Resistor_SMD:R_0805_2012Metric"
 			(at 91.186 124.714 90)
 			(effects
@@
 			)
 		)
-		(property "Footprint" ""
+		(property "Footprint" "LED_SMD:LED_0805_2012Metric"
 			(at 90.17 134.62 0)
 			(effects
@@
 			)
 		)
-		(property "Footprint" ""
+		(property "Footprint" "Capacitor_SMD:C_0805_2012Metric"
 			(at 97.4852 86.36 0)
 			(effects
@@
 			)
 		)
-		(property "Footprint" ""
+		(property "Footprint" "UTSVT_Connectors:Molex_MicroFit3.0_1x2xP3.00mm_PolarizingPeg_Vertical"
 			(at 161.29 100.33 0)
 			(effects
@@
 			)
 		)
-		(property "Footprint" ""
+		(property "Footprint" "Resistor_SMD:R_0805_2012Metric"
 			(at 122.174 62.484 90)
 			(effects
@@
 			)
 		)
-		(property "Footprint" ""
+		(property "Footprint" "UTSVT_Connectors:Molex_MicroFit3.0_1x2xP3.00mm_PolarizingPeg_Vertical"
 			(at 161.29 78.74 0)
 			(effects
@@
 			)
 		)
-		(property "Footprint" ""
+		(property "Footprint" "Resistor_SMD:R_0805_2012Metric"
 			(at 117.856 68.834 90)
 			(effects
@@
 			)
 		)
-		(property "Footprint" ""
+		(property "Footprint" "Diode_SMD:D_0805_2012Metric"
 			(at 171.45 101.6 0)
 			(effects

Commit message: Finished I think :)
Connections:
- net 12V: now also D1.1 (K), D2.1 (K), D3.1 (K), D4.1 (K), J1.2 (Pin_2), J2.2 (Pin_2), J3.2 (Pin_2), J4.2 (Pin_2)
- net FanIn1: no longer R1.1
- net FanIn2: no longer R3.1
- net FanIn3: no longer R5.1
- net FanIn4: no longer R7.1
- net GND: now also Q1.2 (S), Q2.2 (S), Q3.2 (S), Q4.2 (S)
- net at Q1.1 (G), R2.2: now also R1.1
- net at Q4.1 (G), R8.2: now also R7.1
- net at Q2.1 (G), R4.2: now also R3.1
- net at Q3.1 (G), R6.2: now also R5.1
- removed net FanOut1: D1.1 (K), J1.2 (Pin_2), Q1.2 (S)
- removed net FanOut2: D2.1 (K), J2.2 (Pin_2), Q2.2 (S)
- removed net FanOut3: D3.1 (K), J3.2 (Pin_2), Q3.2 (S)
- removed net FanOut4: D4.1 (K), J4.2 (Pin_2), Q4.2 (S)
Other:
- moved on the sheet: R1, R3, R5, R7

Commit message: r pt 2
Other:
- note added: "r"
Changed lines of the file:
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@@
+		)
+	)
+	(text "r\n"
+		(exclude_from_sim no)
+		(at 64.008 92.71 0)
+		(effects
+			(font
+				(size 1.27 1.27)
+			)
 		)
 	)
