File: PCB/FanBoardPCB/FanBoardPCB.kicad_sch (KiCad schematic)
At the start: 4 parts, among them J6 Conn_02x03_Counter_Clockwise

Commit message: This is what I changed
Parts:
- removed C1, C2: C, Capacitor_SMD:C_0805_2012Metric, symbol Device:C
- removed D5: LED, LED_SMD:LED_0805_2012Metric, symbol Device:LED
- removed J6: Conn_02x03_Counter_Clockwise, Connector_Molex:Molex_Micro-Fit_3.0_43045-0612_2x03_P3.00mm_Vertical, symbol Connector_Generic:Conn_02x03_Counter_Clockwise
- added C3, C4: 100 uF, Capacitor_SMD:C_0805_2012Metric, symbol Device:C_Small
- added D6: LED, LED_SMD:LED_0805_2012Metric, symbol Device:LED
- added H1, H2, H3, H4: MountingHole, MountingHole:MountingHole_3mm, symbol Mechanical:MountingHole
- added J5: Fan Board, Connector_Molex:Molex_Micro-Fit_3.0_43045-0612_2x03_P3.00mm_Vertical, symbol Connector_Generic:Conn_02x03_Counter_Clockwise
- added R9: 100k, Resistor_SMD:R_0805_2012Metric, symbol Device:R
Connections:
- net +12V: now also C3.1, C4.2, J5.1 (Pin_1), R9.1
- net Fan2/Fan2: now also J5.3 (Pin_3)
- net Fan3/Fan3: now also J5.4 (Pin_4)
- net Fan4/Fan4: now also J5.5 (Pin_5)
- net GNDPWR: now also C3.2, C4.1
- new net: D6.1 (K), R9.2
- new net: D6.2 (A), J5.6 (Pin_6)
- new net Fan1/poop: J5.2 (Pin_2)
Other:
- sheet Fan1: file untitled.kicad_sch -> fan1.kicad_sch
- sheet Fan1 ports: added poop; removed Fan1
- sheet Fan2: file Fan2.kicad_sch -> untitled.kicad_sch
- sheet Fan3: file Fan3.kicad_sch -> fan3.kicad_sch
- sheet Fan4: file fan4.kicad_sch -> Fan4.kicad_sch
